Commit message: Default not move window, modified husky camera

File: realenv/core/physics/models/husky.urdf (robot description, URDF)
Before this commit: robot husky_robot, 12 links, 11 joints
Joints:
- joint eyes_joint: origin xyz=0.19 0 0.149 rpy=0 0 0 -> xyz=-0.4 0 0.149 rpy=0 0 0

Commit message: new husky model

File: realenv/core/physics/models/husky.urdf (robot description, URDF)
Before this commit: robot husky_robot, 12 links, 11 joints
Links:
- added link top_bumper_link; collision mesh filename=husky_meshes/bumper.stl; visual mesh filename=husky_meshes/bumper.stl
- link eyes: geometry collision sphere radius=0.08; visual cylinder length=0.02 radius=0.03
- link front_bumper_link: geometry collision mesh filename=husky_meshes/bumper.stl; visual mesh filename=husky_meshes/bumper.stl
- link rear_bumper_link: geometry collision mesh filename=husky_meshes/bumper.stl; visual mesh filename=husky_meshes/bumper.stl
Joints:
- added joint top_bumper: type fixed, parent base_link, child top_bumper_link, origin xyz=0 0 0.27 rpy=0 -1.57 0

Commit message: update

File: realenv/core/physics/models/husky.urdf (robot description, URDF)
Before this commit: robot husky_robot, 13 links, 12 joints
Links:
- removed link husky_robot
- link eyes: mass None -> 0
- link front_bumper_link: mass None -> 0
- link imu_link: mass None -> 0
- link rear_bumper_link: mass None -> 0
- link top_bumper_link: mass None -> 0
- link top_plate_link: mass None -> 0
- link user_rail_link: mass None -> 0
Joints:
- removed joint chassis_joint

Commit message: Husky navigate debug: bigger glass shell, constant reward when close to target

File: realenv/core/physics/models/husky.urdf (robot description, URDF)
Before this commit: robot husky_robot, 12 links, 11 joints
Links:
- link eyes: geometry collision sphere radius=0.18; visual cylinder length=0.02 radius=0.03

Commit message: Included new ppo2 from baseline

File: realenv/core/physics/models/husky.urdf (robot description, URDF)
Before this commit: robot husky_robot, 12 links, 11 joints
Links:
- link eyes: geometry collision sphere radius=0.4; visual cylinder length=0.02 radius=0.03

Commit message: New husky high camera model

File: realenv/core/physics/models/husky.urdf (robot description, URDF)
Before this commit: robot husky_robot, 12 links, 11 joints
Links:
- link base_link: mass 30.455 -> 90.455

Commit message: Husky too heavy makes it hard to train

File: realenv/core/physics/models/husky.urdf (robot description, URDF)
Before this commit: robot husky_robot, 12 links, 11 joints
Links:
- link base_link: mass 90.455 -> 30.455

File: realenv/core/physics/models/husky_high.urdf (robot description, URDF)
Before this commit: robot husky_robot, 12 links, 11 joints
Links:
- link base_link: mass 90.455 -> 50.455
Joints:
- joint eyes_joint: origin xyz=-0.4 0 2.525 rpy=0 0 0 -> xyz=-0.4 0 2.5 rpy=0 0 0
