Commit message: Remove robot eye offset value

File: examples/ros/gibson-ros/turtlebot/turtlebot.urdf (robot description, URDF)
Before this commit: robot turtlebot, 34 links, 33 joints
Joints:
- joint camera_joint: origin xyz=-0.031 0.0125 -0.016 rpy=0 0 0 -> xyz=-0.031 0.0125 -0.016 rpy=1.57 0 -1.57
