Commit message: fix turtlebot

File: gibson/assets/models/turtlebot/turtlebot.urdf (robot description, URDF)
Before this commit: robot turtlebot, 35 links, 34 joints
Links:
- removed link base_footprint
- link base_link: geometry collision cylinder length=0.10938 radius=0.176; visual mesh filename=turtlebot/kobuki_description/meshes/main_body.dae
- link kinect_camera: geometry collision box size=0.07271 0.27794 0.073; visual mesh filename=turtlebot/turtlebot_description/meshes/sensors/kinect.dae
- link plate_bottom_link: geometry collision box size=0.26727 0.340 0.006; visual mesh filename=turtlebot/turtlebot_description/meshes/stacks/hexagons/plat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
- link plate_middle_link: geometry collision box size=0.28727 0.340 0.006; visual mesh filename=turtlebot/turtlebot_description/meshes/stacks/hexagons/plat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
- link plate_top_link: geometry collision box size=0.28727 0.340 0.006; visual mesh filename=turtlebot/turtlebot_description/meshes/stacks/hexagons/plat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
- link pole_bottom_0_link: geometry collision cylinder length=0.0492 radius=.006; visual mesh filename=turtlebot/turtlebot_description/meshes/stacks/hexagons/pole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
- link pole_bottom_1_link: geometry collision cylinder length=0.0492 radius=.006; visual mesh filename=turtlebot/turtlebot_description/meshes/stacks/hexagons/pole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
- link pole_bottom_2_link: geometry collision cylinder length=0.0492 radius=.006; visual mesh filename=turtlebot/turtlebot_description/meshes/stacks/hexagons/pole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
- link pole_bottom_3_link: geometry collision cylinder length=0.0492 radius=.006; visual mesh filename=turtlebot/turtlebot_description/meshes/stacks/hexagons/pole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
- link pole_bottom_4_link: geometry collision cylinder length=0.0492 radius=.006; visual mesh filename=turtlebot/turtlebot_description/meshes/stacks/hexagons/pole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
- link pole_bottom_5_link: geometry collision cylinder length=0.0492 radius=.006; visual mesh filename=turtlebot/turtlebot_description/meshes/stacks/hexagons/pole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
- link pole_kinect_0_link: geometry collision cylinder length=0.0936 radius=0.006; visual mesh filename=turtlebot/turtlebot_description/meshes/stacks/hexagons/pole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
- link pole_kinect_1_link: geometry collision cylinder length=0.0936 radius=0.006; visual mesh filename=turtlebot/turtlebot_description/meshes/stacks/hexagons/pole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
- link pole_middle_0_link: geometry collision cylinder length=0.0608 radius=.006; visual mesh filename=turtlebot/turtlebot_description/meshes/stacks/hexagons/pole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
- link pole_middle_1_link: geometry collision cylinder length=0.0608 radius=.006; visual mesh filename=turtlebot/turtlebot_description/meshes/stacks/hexagons/pole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
- link pole_middle_2_link: geometry collision cylinder length=0.0608 radius=.006; visual mesh filename=turtlebot/turtlebot_description/meshes/stacks/hexagons/pole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
- link pole_middle_3_link: geometry collision cylinder length=0.0608 radius=.006; visual mesh filename=turtlebot/turtlebot_description/meshes/stacks/hexagons/pole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
- link pole_top_0_link: geometry collision cylinder length=0.2032 radius=.006; visual mesh filename=turtlebot/turtlebot_description/meshes/stacks/hexagons/pole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
- link pole_top_1_link: geometry collision cylinder length=0.2032 radius=.006; visual mesh filename=turtlebot/turtlebot_description/meshes/stacks/hexagons/pole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
- link pole_top_2_link: geometry collision cylinder length=0.2032 radius=.006; visual mesh filename=turtlebot/turtlebot_description/meshes/stacks/hexagons/pole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
- link pole_top_3_link: geometry collision cylinder length=0.2032 radius=.006; visual mesh filename=turtlebot/turtlebot_description/meshes/stacks/hexagons/pole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
- link wheel_left_link: geometry collision cylinder length=0.0206 radius=0.0352; visual mesh filename=turtlebot/kobuki_description/meshes/wheel.dae
- link wheel_right_link: geometry collision cylinder length=0.0206 radius=0.0350; visual mesh filename=turtlebot/kobuki_description/meshes/wheel.dae
Joints:
- removed joint base_joint
- joint eye_joint: origin xyz=0 0.025 0 rpy=0 0 0 -> xyz=0 0.025 0 rpy=1.57079632679 0 -1.57079632679; parent camera_rgb_optical_frame -> kinect_camera

File: gibson/assets/models/turtlebot/turtlebot_description/turtlebot.urdf (robot description, URDF)
Before this commit: robot turtlebot, 35 links, 34 joints
Links:
- removed link eyes
- removed link kinect_camera
- added link camera_link, mass 0.001; collision box size=0.07271 0.27794 0.073; visual mesh filename=package://turtlebot_description/meshes/sensors/kinect.dae
- link base_link: geometry collision cylinder length=0.10938 radius=0.176; visual mesh filename=package://kobuki_description/meshes/main_body.dae
- link plate_bottom_link: geometry collision box size=0.26727 0.340 0.006; visual mesh filename=package://turtlebot_description/meshes/stacks/hexagons/plat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
- link plate_middle_link: geometry collision box size=0.28727 0.340 0.006; visual mesh filename=package://turtlebot_description/meshes/stacks/hexagons/plat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
- link plate_top_link: geometry collision box size=0.28727 0.340 0.006; visual mesh filename=package://turtlebot_description/meshes/stacks/hexagons/plat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
- link pole_bottom_0_link: geometry collision cylinder length=0.0492 radius=.006; visual mesh filename=package://turtlebot_description/meshes/stacks/hexagons/pole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
- link pole_bottom_1_link: geometry collision cylinder length=0.0492 radius=.006; visual mesh filename=package://turtlebot_description/meshes/stacks/hexagons/pole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
- link pole_bottom_2_link: geometry collision cylinder length=0.0492 radius=.006; visual mesh filename=package://turtlebot_description/meshes/stacks/hexagons/pole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
- link pole_bottom_3_link: geometry collision cylinder length=0.0492 radius=.006; visual mesh filename=package://turtlebot_description/meshes/stacks/hexagons/pole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
- link pole_bottom_4_link: geometry collision cylinder length=0.0492 radius=.006; visual mesh filename=package://turtlebot_description/meshes/stacks/hexagons/pole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
- link pole_bottom_5_link: geometry collision cylinder length=0.0492 radius=.006; visual mesh filename=package://turtlebot_description/meshes/stacks/hexagons/pole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
- link pole_kinect_0_link: geometry collision cylinder length=0.0936 radius=0.006; visual mesh filename=package://turtlebot_description/meshes/stacks/hexagons/pole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
- link pole_kinect_1_link: geometry collision cylinder length=0.0936 radius=0.006; visual mesh filename=package://turtlebot_description/meshes/stacks/hexagons/pole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
- link pole_middle_0_link: geometry collision cylinder length=0.0608 radius=.006; visual mesh filename=package://turtlebot_description/meshes/stacks/hexagons/pole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
- link pole_middle_1_link: geometry collision cylinder length=0.0608 radius=.006; visual mesh filename=package://turtlebot_description/meshes/stacks/hexagons/pole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
- link pole_middle_2_link: geometry collision cylinder length=0.0608 radius=.006; visual mesh filename=package://turtlebot_description/meshes/stacks/hexagons/pole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
- link pole_middle_3_link: geometry collision cylinder length=0.0608 radius=.006; visual mesh filename=package://turtlebot_description/meshes/stacks/hexagons/pole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
- link pole_top_0_link: geometry collision cylinder length=0.2032 radius=.006; visual mesh filename=package://turtlebot_description/meshes/stacks/hexagons/pole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
- link pole_top_1_link: geometry collision cylinder length=0.2032 radius=.006; visual mesh filename=package://turtlebot_description/meshes/stacks/hexagons/pole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
- link pole_top_2_link: geometry collision cylinder length=0.2032 radius=.006; visual mesh filename=package://turtlebot_description/meshes/stacks/hexagons/pole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
- link pole_top_3_link: geometry collision cylinder length=0.2032 radius=.006; visual mesh filename=package://turtlebot_description/meshes/stacks/hexagons/pole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
- link wheel_left_link: mass 0.1 -> 0.01; geometry collision cylinder length=0.0206 radius=0.0352; visual mesh filename=package://kobuki_description/meshes/wheel.dae
- link wheel_right_link: mass 0.1 -> 0.01; geometry collision cylinder length=0.0206 radius=0.0350; visual mesh filename=package://kobuki_description/meshes/wheel.dae
Joints:
- removed joint eye_joint
- joint camera_joint: child kinect_camera -> camera_link
