Commit message: modified turtlebot and husky URDF to increase camera height

File: gibson/assets/models/husky.urdf (robot description, URDF)
Before this commit: robot husky_robot, 12 links, 11 joints
Joints:
- joint eyes_joint: origin xyz=0.4 0 0.149 rpy=1.57 0 -1.57 -> xyz=0.4 0 1.0 rpy=1.57 0 -1.57

File: gibson/assets/models/turtlebot/turtlebot.urdf (robot description, URDF)
Before this commit: robot turtlebot, 34 links, 33 joints
Joints:
- joint camera_rgb_joint: origin xyz=-0.087 -0.0125 0.287 rpy=0 0 0 -> xyz=-0.087 -0.0125 1.000 rpy=0 0 0

File: gibson/assets/models/turtlebot/turtlebot_description/turtlebot.urdf (robot description, URDF)
Before this commit: robot turtlebot, 34 links, 33 joints
Joints:
- joint camera_rgb_joint: origin xyz=-0.087 -0.0125 0.287 rpy=0 0 0 -> xyz=-0.087 -0.0125 1.000 rpy=0 0 0

Commit message: restored default robot models

File: gibson/assets/models/husky.urdf (robot description, URDF)
Before this commit: robot husky_robot, 12 links, 11 joints
Joints:
- joint eyes_joint: origin xyz=0.4 0 1.0 rpy=1.57 0 -1.57 -> xyz=0.4 0 0.149 rpy=1.57 0 -1.57

File: gibson/assets/models/turtlebot/turtlebot.urdf (robot description, URDF)
Before this commit: robot turtlebot, 34 links, 33 joints
Joints:
- joint camera_rgb_joint: origin xyz=-0.087 -0.0125 1.000 rpy=0 0 0 -> xyz=-0.087 -0.0125 0.287 rpy=0 0 0

File: gibson/assets/models/turtlebot/turtlebot_description/turtlebot.urdf (robot description, URDF)
Before this commit: robot turtlebot, 34 links, 33 joints
Joints:
- joint camera_rgb_joint: origin xyz=-0.087 -0.0125 1.000 rpy=0 0 0 -> xyz=-0.087 -0.0125 0.287 rpy=0 0 0
